File: pcb/wrx/wrx.ADC.sch (KiCad schematic (older format))
At the start: 59 parts, among them J1 TB_2, U401 LTC2248, U402 65.360 MHz, U404 LP5907 3.3V 250mA, U405 LTC6401-20, U406 NC7SZ126

Commit message: big update to, and reorg of, PCB design files
The active antenna PCB has been split-out from the Beagle cape KiCAD
files. This was done so separate BOMs could be more easily created.
Parts:
- removed U402: 65.360 MHz, wrx-VCXO, symbol VCXO
- removed U406: NC7SZ126, wrx-SC70_5, symbol LOGIC_126_BUF
- added C417: 10n, wrx-SM0402, symbol C
- added J2: DNL BNC, wrx-BNC_SMA_EM, symbol COAX_CONN_3P
- added J5: DNL U.FL, wrx-U.FL, symbol COAX_CONN_3P
- added TP401: TEST_POINT, wrx-TP_600, symbol TEST_POINT
- added TP402: TEST_POINT, wrx-TP_VIA_600, symbol TEST_POINT
- added U402: 66.6666 MHz, wrx-XO, symbol XO
- added U403, U406: NC7SZ125, wrx-SC70_5, symbol LOGIC_125_BUF
- added Z401: TVS 3.3V, wrx-SOD323, symbol TVS
- C401, C404: value 56p -> 56p/100
- C402, C403: value 160p -> 160p/50
- C405: value 1n -> 1n/100; footprint wrx-SM0402 -> wrx-SM0805
- C406: value 470n -> 470n/100; footprint wrx-SM0402 -> wrx-SM1206
- J1: footprint wrx-TERM_BLOCK_2 -> wrx-TB_2P_2_54MM
- Z402: renamed from Z401; value TVS 40V -> TVS 3.3V; footprint wrx-SM0402 -> wrx-SOD323
Connections:
- net labels added: AEXT, AXO, ECLK
- net labels removed: VCXO
- wire segments 229 -> 250
- no-connect marks 6 -> 4
Other:
- note added: "using BNC_SMA_EM\nfootprint to allow\nSMA connector option"
- moved on the sheet: C401, C402, C403, C404, C405, C406, C425, J1, L401, L402, L403, L404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
