File: pcb/wrx/wrx.power_supplies.sch (KiCad schematic (older format))
At the start: 13 parts, among them U701 LMR10530Y 1.0V 3A, U702 LP5907 1.8V 250mA

Commit message: big update to, and reorg of, PCB design files
The active antenna PCB has been split-out from the Beagle cape KiCAD
files. This was done so separate BOMs could be more easily created.
Parts:
- added TP701, TP702: TEST_POINT, wrx-TP_600, symbol TEST_POINT
Connections:
- net 1.0: now also TP701.1
- net 1.8: now also TP702.1
Changed lines of the file:
@@
-EESchema Schematic File Version 2  date Sunday, May 10, 2015 01:16:43 PM
+EESchema Schematic File Version 2  date Friday, July 17, 2015 09:41:48 AM
 LIBS:wrx
 LIBS:wrx-cache
@@
 encoding utf-8
 Sheet 7 7
-Title "Power Supplies"
-Date "7 may 2015"
-Rev ""
-Comp ""
+Title "WRX Prototype v0.1"
+Date "16 jul 2015"
+Rev "0.1"
+Comp "Point Reyes Ventures, LLC"
 Comment1 ""
 Comment2 ""
@@
 $EndDescr
 $Comp
-L GND #PWR0113
+L GND #PWR0117
 U 1 1 50832A56
 P 4300 4300
-F 0 "#PWR0113" H 4300 4300 30  0001 C CNN
+F 0 "#PWR0117" H 4300 4300 30  0001 C CNN
 F 1 "GND" H 4300 4230 30  0001 C CNN
 F 2 "" H 4300 4300 60  0001 C CNN
@@
 	8850 2950 8850 2900
 $Comp
-L GND #PWR0114
+L GND #PWR0118
 U 1 1 52C1F4EA
 P 5800 2300
-F 0 "#PWR0114" H 5800 2300 30  0001 C CNN
+F 0 "#PWR0118" H 5800 2300 30  0001 C CNN
 F 1 "GND" H 5800 2230 30  0001 C CNN
 F 2 "" H 5800 2300 60  0001 C CNN
@@
 Connection ~ 3000 2950
 $Comp
-L 5V #PWR0115
+L 5V #PWR0119
 U 1 1 52C20291
 P 2200 2900
-F 0 "#PWR0115" H 2200 2990 20  0001 C CNN
+F 0 "#PWR0119" H 2200 2990 20  0001 C CNN
 F 1 "5V" H 2200 2990 30  0000 C CNN
 F 2 "~" H 2200 2900 60  0000 C CNN
@@
 SW2
 $Comp
-L 5V #PWR0116
+L 5V #PWR0120
 U 1 1 54E56ABD
 P 6650 5650
-F 0 "#PWR0116" H 6650 5740 20  0001 C CNN
+F 0 "#PWR0120" H 6650 5740 20  0001 C CNN
 F 1 "5V" H 6650 5740 30  0000 C CNN
 F 2 "~" H 6650 5650 60  0000 C CNN
@@
 	6650 5700 6750 5700
 Wire Wire Line
-	9150 5700 9250 5700
+	9150 5700 9450 5700
 Wire Wire Line
 	9250 5700 9250 5650
 $Comp
-L GND #PWR0117
+L GND #PWR0121
 U 1 1 54E56ACD
 P 7850 6500
-F 0 "#PWR0117" H 7850 6500 30  0001 C CNN
+F 0 "#PWR0121" H 7850 6500 30  0001 C CNN
 F 1 "GND" H 7850 6430 30  0001 C CNN
 F 2 "~" H 7850 6500 60  0000 C CNN
@@
 	7850 6400 7850 6500
 $Comp
-L 1.8 #PWR0118
+L 1.8 #PWR0122
 U 1 1 54E56AE2
 P 9250 5650
-F 0 "#PWR0118" H 9250 5610 30  0001 C CNN
+F 0 "#PWR0122" H 9250 5610 30  0001 C CNN
 F 1 "1.8" H 9250 5760 30  0000 C CNN
 F 2 "~" H 9250 5650 60  0000 C CNN
@@
 $EndComp
 $Comp
-L 1.0 #PWR0119
+L 1.0 #PWR0123
 U 1 1 54E552B4
 P 8850 2900
-F 0 "#PWR0119" H 8850 2860 30  0001 C CNN
+F 0 "#PWR0123" H 8850 2860 30  0001 C CNN
 F 1 "1.0" H 8850 3010 30  0000 C CNN
 F 2 "~" H 8850 2900 60  0000 C CNN
@@
 $EndComp
 $Comp
-L PWR_DRV #PWR0120
+L PWR_DRV #PWR0124
 U 1 1 54E9A12C
 P 8550 2950
-F 0 "#PWR0120" H 8500 3050 40  0001 C CNN
+F 0 "#PWR0124" H 8500 3050 40  0001 C CNN
 F 1 "PWR_DRV" H 8500 2850 40  0001 C CNN
 F 2 "~" H 8550 2950 60  0000 C CNN
@@
 	6650 6200 6650 6250
 $Comp
-L GND #PWR0121
+L GND #PWR0125
 U 1 1 54F3EFD6
 P 6650 6250
-F 0 "#PWR0121" H 6650 6250 30  0001 C CNN
+F 0 "#PWR0125" H 6650 6250 30  0001 C CNN
 F 1 "GND" H 6650 6180 30  0001 C CNN
 F 2 "~" H 6650 6250 60  0000 C CNN
@@
 	9150 6200 9150 6250
 $Comp
-L GND #PWR0122
+L GND #PWR0126
 U 1 1 54F3F01F
 P 9150 6250
-F 0 "#PWR0122" H 9150 6250 30  0001 C CNN
+F 0 "#PWR0126" H 9150 6250 30  0001 C CNN
 F 1 "GND" H 9150 6180 30  0001 C CNN
 F 2 "~" H 9150 6250 60  0000 C CNN
@@
 	2300 4200 8100 4200
 Wire Wire Line
-	8550 2950 8850 2950
+	8550 2950 9050 2950
 Text Label 8600 2950 0    60   ~ 0
 SW2
 $Comp
-L 5V #PWR0123
+L 5V #PWR0127
 U 1 1 55274AE8
 P 8250 6450
-F 0 "#PWR0123" H 8250 6540 20  0001 C CNN
+F 0 "#PWR0127" H 8250 6540 20  0001 C CNN
 F 1 "5V" H 8250 6540 30  0000 C CNN
 F 2 "~" H 8250 6450 60  0000 C CNN
@@
 $EndComp
 $Comp
-L 1.8 #PWR0124
+L 1.8 #PWR0128
 U 1 1 552EE5D9
 P 7450 6450
-F 0 "#PWR0124" H 7450 6410 30  0001 C CNN
+F 0 "#PWR0128" H 7450 6410 30  0001 C CNN
 F 1 "1.8" H 7450 6560 30  0000 C CNN
 F 2 "~" H 7450 6450 60  0000 C CNN
@@
 Wire Wire Line
 	7700 3600 7700 3450
+$Comp
+L TEST_POINT TP701
+U 1 1 556D0342
+P 9050 2800
+F 0 "TP701" H 9050 2950 60  0000 C CNN
+F 1 "TEST_POINT" H 9050 2600 60  0001 C CNN
+F 2 "wrx-TP_600" H 9050 2800 60  0001 C CNN
+F 3 "~" H 9050 2800 60  0000 C CNN
+	1    9050 2800
+	1    0    0    -1
+$EndComp
+Wire Wire Line
+	9050 2950 9050 2900
+Connection ~ 8850 2950
+$Comp
+L TEST_POINT TP702
+U 1 1 556D03DB
+P 9450 5550
+F 0 "TP702" H 9450 5700 60  0000 C CNN
+F 1 "TEST_POINT" H 9450 5350 60  0001 C CNN
+F 2 "wrx-TP_600" H 9450 5550 60  0001 C CNN
+F 3 "~" H 9450 5550 60  0000 C CNN
+	1    9450 5550
+	1    0    0    -1
+$EndComp
+Wire Wire Line
+	9450 5700 9450 5650
+Connection ~ 9250 5700
 $EndSCHEMATC
