File: pcb/active_ant_opts/ant.Mini_Whip.sch (KiCad schematic (older format))
At the start: 46 parts, among them J10 TB_2, J11 DNL RJ45, J12 DNL TB_2, J13 EARTH GROUND, Q501 J310, Q505 BFG35, T503 CMC 4.7 mH, T504 DNL T1-6, U501 TPS7A4501

Commit message: big update supporting first PCB fab
Big changes to Artix-7 A35 FPGA on first PCB fab.
Renaming project to "KiwiSDR".
New thread priority scheme.
New eCPU stack checking code.
Many performance improvements.
GPS timing now adjusts XO frequency.
New SPI transfer integrity checking code.
Improved event recording debug facility.
Parts:
- C501, C502, C506, C521: footprint wrx-SM1206 -> kiwi-SM1206
- C509, C510, C511, C512, C513, C514, C515, C520, C522, C523, C526, L501, L502, L503, L507, R502, R505, R507, R510, R511, R512, R514, R517, R519, R520, R521, R522, R523, R524, R525: footprint wrx-SM0805 -> kiwi-SM0805
- G501, G502: footprint wrx-GDT -> kiwi-GDT
- J10, J12: footprint wrx-TERM_BLOCK_2 -> kiwi-TERM_BLOCK_2
- J11: footprint wrx-RJ45_8 -> kiwi-RJ45_8
- J13: footprint wrx-SCREW_HOLE_#8 -> kiwi-SCREW_HOLE_#8
- L506: footprint wrx-SM1812 -> kiwi-SM1812
- Q501: footprint wrx-SOT23_DGS -> kiwi-SOT23_DGS
- Q505: footprint wrx-SOT233_BCE -> kiwi-SOT233_BCE
- T503: footprint wrx-CMC -> kiwi-CMC
- T504: footprint wrx-MCL_KK81 -> kiwi-MCL_KK81
- U501: footprint wrx-SOT232_6 -> kiwi-SOT232_6
