File: pcb/active_ant_opts/ant.inj_CAT5.sch (KiCad schematic (older format))
At the start: 32 parts, among them J20 TB_2, J21 TB_2, J22 TB_2, J23 RJ45, J24 TB_2, T201 CMC 4.7 mH, T202 CMC 4.7 mH, T203 T1-6, U201 LM2941

Commit message: big update supporting first PCB fab
Big changes to Artix-7 A35 FPGA on first PCB fab.
Renaming project to "KiwiSDR".
New thread priority scheme.
New eCPU stack checking code.
Many performance improvements.
GPS timing now adjusts XO frequency.
New SPI transfer integrity checking code.
Improved event recording debug facility.
Parts:
- C201, C203, C214: footprint wrx-SM1206 -> kiwi-SM1206
- C204, C205, C206, C207, C208, D202, R201, R202, R203, R204, R205, R206, R207: footprint wrx-SM0805 -> kiwi-SM0805
- C209: footprint wrx-CAP_10x10 -> kiwi-CAP_10x10
- C210: footprint wrx-CAP_D -> kiwi-CAP_D
- C211, C212: footprint wrx-SM0603 -> kiwi-SM0603
- D201: footprint wrx-TO269_AA -> kiwi-TO269_AA
- F201, F202: footprint wrx-SM1812 -> kiwi-SM1812
- J20, J21, J22, J24: footprint wrx-TERM_BLOCK_2 -> kiwi-TERM_BLOCK_2
- J23: footprint wrx-RJ45_8 -> kiwi-RJ45_8
- T201, T202: footprint wrx-CMC -> kiwi-CMC
- T203: footprint wrx-MCL_KK81 -> kiwi-MCL_KK81
- U201: footprint wrx-TO263 -> kiwi-TO263
Changed lines of the file:
@@
 EESchema Schematic File Version 2  date Friday, March 20, 2015 01:09:53 PM
-LIBS:wrx
+LIBS:kiwi
 EELAYER 27 0
 EELAYER END
@@
 F 0 "C212" H 6550 4650 40  0000 L CNN
 F 1 "1u" H 6556 4465 40  0000 L CNN
-F 2 "wrx-SM0603" H 6588 4400 30  0001 C CNN
+F 2 "kiwi-SM0603" H 6588 4400 30  0001 C CNN
 F 3 "~" H 6550 4550 60  0000 C CNN
 	1    6550 4550
@@
 F 0 "J22" H 15800 4950 50  0000 C CNN
 F 1 "TB_2" H 15800 4150 50  0000 C CNN
-F 2 "wrx-TERM_BLOCK_2" H 15800 4550 60  0001 C CNN
+F 2 "kiwi-TERM_BLOCK_2" H 15800 4550 60  0001 C CNN
 F 3 "~" H 15800 4550 60  0000 C CNN
 	1    15800 4550
@@
 F 0 "R201" V 11030 4550 40  0000 C CNN
 F 1 "680R" V 10957 4551 40  0000 C CNN
-F 2 "wrx-SM0805" V 10880 4550 30  0001 C CNN
+F 2 "kiwi-SM0805" V 10880 4550 30  0001 C CNN
 F 3 "~" H 10950 4550 30  0000 C CNN
 	1    10950 4550
@@
 F 0 "J20" H 5700 6100 50  0000 C CNN
 F 1 "TB_2" H 5700 6000 50  0000 C CNN
-F 2 "wrx-TERM_BLOCK_2" H 5450 6000 60  0001 C CNN
+F 2 "kiwi-TERM_BLOCK_2" H 5450 6000 60  0001 C CNN
 F 3 "~" H 5450 6000 60  0000 C CNN
 	1    5450 6000
@@
 F 0 "D201" H 11900 4550 40  0000 C CNN
 F 1 "BR 0.5A 400V" H 12350 4550 40  0000 C CNN
-F 2 "wrx-TO269_AA" V 11980 4300 30  0001 C CNN
+F 2 "kiwi-TO269_AA" V 11980 4300 30  0001 C CNN
 F 3 "~" H 12050 4300 30  0000 C CNN
 	1    12050 4550
@@
 F 0 "C205" V 12050 4000 40  0000 L CNN
 F 1 "100n/100" V 12050 3600 40  0000 L CNN
-F 2 "wrx-SM0805" H 12038 3800 30  0001 C CNN
+F 2 "kiwi-SM0805" H 12038 3800 30  0001 C CNN
 F 3 "~" H 12000 3950 60  0000 C CNN
 	1    12000 3950
@@
 F 0 "C206" V 12050 5200 40  0000 L CNN
 F 1 "100n/100" V 12050 4800 40  0000 L CNN
-F 2 "wrx-SM0805" H 12038 5000 30  0001 C CNN
+F 2 "kiwi-SM0805" H 12038 5000 30  0001 C CNN
 F 3 "~" H 12000 5150 60  0000 C CNN
 	1    12000 5150
@@
 F 0 "C204" V 12050 3400 40  0000 L CNN
 F 1 "100n/100" V 12050 3000 40  0000 L CNN
-F 2 "wrx-SM0805" H 12038 3200 30  0001 C CNN
+F 2 "kiwi-SM0805" H 12038 3200 30  0001 C CNN
 F 3 "~" H 12000 3350 60  0000 C CNN
 	1    12000 3350
@@
 F 0 "C207" V 12050 5800 40  0000 L CNN
 F 1 "100n/100" V 12050 5400 40  0000 L CNN
-F 2 "wrx-SM0805" H 12038 5600 30  0001 C CNN
+F 2 "kiwi-SM0805" H 12038 5600 30  0001 C CNN
 F 3 "~" H 12000 5750 60  0000 C CNN
 	1    12000 5750
@@
 F 0 "C208" H 10400 4650 40  0000 L CNN
 F 1 "100n/100" V 10750 4400 40  0000 L CNN
-F 2 "wrx-SM0805" H 10638 4400 30  0001 C CNN
+F 2 "kiwi-SM0805" H 10638 4400 30  0001 C CNN
 F 3 "~" H 10600 4550 60  0000 C CNN
 	1    10600 4550
@@
 F 0 "R202" V 8280 4650 40  0000 C CNN
 F 1 "11K5" V 8207 4651 40  0000 C CNN
-F 2 "wrx-SM0805" V 8130 4650 30  0001 C CNN
+F 2 "kiwi-SM0805" V 8130 4650 30  0001 C CNN
 F 3 "~" H 8200 4650 30  0000 C CNN
 	1    8200 4650
@@
 F 0 "R203" V 8280 5350 40  0000 C CNN
 F 1 "1K" V 8207 5351 40  0000 C CNN
-F 2 "wrx-SM0805" V 8130 5350 30  0001 C CNN
+F 2 "kiwi-SM0805" V 8130 5350 30  0001 C CNN
 F 3 "~" H 8200 5350 30  0000 C CNN
 	1    8200 5350
@@
 F 0 "J21" H 1800 6350 50  0000 C CNN
 F 1 "TB_2" H 1800 5600 50  0000 C CNN
-F 2 "wrx-TERM_BLOCK_2" H 1800 6000 60  0001 C CNN
+F 2 "kiwi-TERM_BLOCK_2" H 1800 6000 60  0001 C CNN
 F 3 "~" H 1800 6000 60  0000 C CNN
 	1    1800 6000
@@
 F 0 "C211" H 6800 4650 40  0000 L CNN
 F 1 "1n" H 6806 4465 40  0000 L CNN
-F 2 "wrx-SM0603" H 6838 4400 30  0001 C CNN
+F 2 "kiwi-SM0603" H 6838 4400 30  0001 C CNN
 F 3 "~" H 6800 4550 60  0000 C CNN
 	1    6800 4550
@@
 F 0 "C209" H 10000 4650 40  0000 L CNN
 F 1 "470u/35 EL" H 10000 4450 40  0000 L CNN
-F 2 "wrx-CAP_10x10" H 10000 4550 60  0001 C CNN
+F 2 "kiwi-CAP_10x10" H 10000 4550 60  0001 C CNN
 F 3 "~" H 10000 4550 60  0000 C CNN
 	1    10000 4550
@@
 F 0 "T203" H 3050 6000 50  0000 L BNN
 F 1 "T1-6" H 3600 6000 50  0000 L BNN
-F 2 "wrx-MCL_KK81" H 3450 6000 60  0001 C CNN
+F 2 "kiwi-MCL_KK81" H 3450 6000 60  0001 C CNN
 F 3 "~" H 3450 6000 60  0000 C CNN
 	1    3450 6000
@@
 F 0 "T201" H 5450 4800 50  0000 C BNN
 F 1 "CMC 4.7 mH" H 5450 4200 50  0000 C BNN
-F 2 "wrx-CMC" H 5450 4550 60  0001 C CNN
+F 2 "kiwi-CMC" H 5450 4550 60  0001 C CNN
 F 3 "~" H 5450 4550 60  0000 C CNN
 	1    5450 4550
@@
 F 0 "U201" H 8850 4250 60  0000 C CNN
 F 1 "LM2941" H 8850 4400 60  0000 C CNN
-F 2 "wrx-TO263" H 8800 3900 60  0001 C CNN
+F 2 "kiwi-TO263" H 8800 3900 60  0001 C CNN
 F 3 "~" H 8800 3900 60  0000 C CNN
 	1    8850 4250
@@
 F 0 "J23" V 2050 4750 60  0000 C CNN
 F 1 "RJ45" V 1150 4600 60  0000 C CNN
-F 2 "wrx-RJ45_8" H 1600 4600 60  0001 C CNN
+F 2 "kiwi-RJ45_8" H 1600 4600 60  0001 C CNN
 F 3 "~" H 1600 4600 60  0000 C CNN
 	1    1600 4600
@@
 F 0 "J24" H 2050 3500 50  0000 C CNN
 F 1 "TB_2" H 2150 3600 50  0000 C CNN
-F 2 "wrx-TERM_BLOCK_2" H 1800 3600 60  0001 C CNN
+F 2 "kiwi-TERM_BLOCK_2" H 1800 3600 60  0001 C CNN
 F 3 "~" H 1800 3600 60  0000 C CNN
 	1    1800 3600
@@
 F 0 "F201" H 7450 4350 40  0000 C CNN
 F 1 "PPTC 200 mA" H 7350 4100 40  0000 C CNN
-F 2 "wrx-SM1812" H 7350 4180 30  0001 C CNN
+F 2 "kiwi-SM1812" H 7350 4180 30  0001 C CNN
 F 3 "~" V 7350 4250 30  0000 C CNN
 	1    7350 4250
@@
 F 0 "C203" H 12950 4650 40  0000 L CNN
 F 1 "470n/100" H 12956 4465 40  0000 L CNN
-F 2 "wrx-SM1206" H 12988 4400 30  0001 C CNN
+F 2 "kiwi-SM1206" H 12988 4400 30  0001 C CNN
 F 3 "~" H 12950 4550 60  0000 C CNN
 	1    12950 4550
@@
 F 0 "C210" H 7900 4650 40  0000 L CNN
 F 1 "22u/25 TA" H 7550 4450 40  0000 L CNN
-F 2 "wrx-CAP_D" H 7900 4550 60  0001 C CNN
+F 2 "kiwi-CAP_D" H 7900 4550 60  0001 C CNN
 F 3 "~" H 7900 4550 60  0000 C CNN
 F 4 "ESR 0.1-1R" H 7500 4400 40  0000 L CNN "Field4"
@@
 F 0 "C214" H 9600 4650 40  0000 L CNN
 F 1 "470n/100" H 9606 4465 40  0000 L CNN
-F 2 "wrx-SM1206" H 9638 4400 30  0001 C CNN
+F 2 "kiwi-SM1206" H 9638 4400 30  0001 C CNN
 F 3 "~" H 9600 4550 60  0000 C CNN
 	1    9600 4550
@@
 F 0 "T202" V 14150 4550 50  0000 C BNN
 F 1 "CMC 4.7 mH" H 13900 4200 50  0000 C BNN
-F 2 "wrx-CMC" H 13900 4550 60  0001 C CNN
+F 2 "kiwi-CMC" H 13900 4550 60  0001 C CNN
 F 3 "~" H 13900 4550 60  0000 C CNN
 	1    13900 4550
@@
 F 0 "F202" H 15250 4350 40  0000 C CNN
 F 1 "PPTC 200 mA" H 15150 4100 40  0000 C CNN
-F 2 "wrx-SM1812" H 15150 4180 30  0001 C CNN
+F 2 "kiwi-SM1812" H 15150 4180 30  0001 C CNN
 F 3 "~" V 15150 4250 30  0000 C CNN
 	1    15150 4250
@@
 F 0 "C201" H 13300 4650 40  0000 L CNN
 F 1 "470n/100" H 13306 4465 40  0000 L CNN
-F 2 "wrx-SM1206" H 13338 4400 30  0001 C CNN
+F 2 "kiwi-SM1206" H 13338 4400 30  0001 C CNN
 F 3 "~" H 13300 4550 60  0000 C CNN
 	1    13300 4550
@@
 F 0 "R205" V 12080 3650 40  0000 C CNN
 F 1 "47R" V 12007 3651 40  0000 C CNN
-F 2 "wrx-SM0805" V 11930 3650 30  0001 C CNN
+F 2 "kiwi-SM0805" V 11930 3650 30  0001 C CNN
 F 3 "~" H 12000 3650 30  0000 C CNN
 	1    12000 3650
@@
 F 0 "R204" V 12080 3050 40  0000 C CNN
 F 1 "47R" V 12007 3051 40  0000 C CNN
-F 2 "wrx-SM0805" V 11930 3050 30  0001 C CNN
+F 2 "kiwi-SM0805" V 11930 3050 30  0001 C CNN
 F 3 "~" H 12000 3050 30  0000 C CNN
 	1    12000 3050
@@
 F 0 "R206" V 12080 5450 40  0000 C CNN
 F 1 "47R" V 12007 5451 40  0000 C CNN
-F 2 "wrx-SM0805" V 11930 5450 30  0001 C CNN
+F 2 "kiwi-SM0805" V 11930 5450 30  0001 C CNN
 F 3 "~" H 12000 5450 30  0000 C CNN
 	1    12000 5450
@@
 F 0 "R207" V 12080 6050 40  0000 C CNN
 F 1 "47R" V 12007 6051 40  0000 C CNN
-F 2 "wrx-SM0805" V 11930 6050 30  0001 C CNN
+F 2 "kiwi-SM0805" V 11930 6050 30  0001 C CNN
 F 3 "~" H 12000 6050 30  0000 C CNN
 	1    12000 6050
@@
 F 0 "D202" H 14600 4650 50  0000 C CNN
 F 1 "TVS 25V" H 14600 4400 50  0000 C CNN
-F 2 "wrx-SM0805" H 14550 4450 60  0001 C CNN
+F 2 "kiwi-SM0805" H 14550 4450 60  0001 C CNN
 F 3 "~" H 14550 4450 60  0000 C CNN
 	1    14600 4550
