File: pcb/KiwiSDR/kiwi.ADC.sch (KiCad schematic (older format))
At the start: 66 parts, among them J1 TB_2, J2 DNL BNC, J5 DNL U.FL, U401 LTC2248, U402 66.6666 MHz, U403 NC7SZ125, U404 LP5907 3.3V 250mA, U405 LTC6401-20, U406 NC7SZ125

Commit message: v0.5 PCB with 5V DC input
Parts:
- J2: value DNL BNC -> SMA; footprint kiwi-BNC_SMA_EM -> kiwi-SMA_OPL_EM
Other:
- note removed: "using BNC_SMA_EM\nfootprint to allow\nSMA connector option"
Changed lines of the file:
@@
-EESchema Schematic File Version 2  date Wednesday, January 13, 2016 07:56:48 PM
+EESchema Schematic File Version 2  date Sunday, February 21, 2016 12:56:59 PM
 LIBS:kiwi
+LIBS:kiwi-cache
 EELAYER 27 0
 EELAYER END
@@
 encoding utf-8
 Sheet 2 7
-Title "KiwiSDR Prototype v0.3"
-Date "30 jul 2015"
-Rev "0.3"
-Comp "Point Reyes Ventures, LLC"
+Title "KiwiSDR Prototype, March 2016"
+Date "20 feb 2016"
+Rev "0.5"
+Comp "John Seamons, ZL/KF6VO"
 Comment1 ""
 Comment2 ""
@@
 P 2500 3050
 F 0 "J2" H 2510 3170 60  0000 C CNN
-F 1 "DNL BNC" V 2610 2990 50  0000 C CNN
-F 2 "kiwi-BNC_SMA_EM" H 2500 3050 60  0001 C CNN
+F 1 "SMA" V 2610 2990 50  0000 C CNN
+F 2 "kiwi-SMA_OPL_EM" H 2500 3050 60  0001 C CNN
 F 3 "~" H 2500 3050 60  0000 C CNN
 	1    2500 3050
@@
 Wire Wire Line
 	2650 2800 2650 3050
-Text Notes 2200 3050 2    60   ~ 0
-using BNC_SMA_EM\nfootprint to allow\nSMA connector option
 Wire Wire Line
 	8800 2800 9700 2800
