File: pcb/active_antenna/ant.kicad_pcb (KiCad board)
At the start: 2 copper layers, 300 x 155 mm, 130 parts, among them J10 TB_2, J11 DNL RJ45, J12 DNL TB_2, J13 EARTH GROUND, J14 DNL BNC, J20 TB_2, J21 TB_2, J22 DC JACK 2.1MM, J23 DNL RJ45, J24 DNL TB_2, J25 DNL BNC, J26 DNL BNC, Q501 J310, Q502 DNL J271, Q503 DNL BFG31, Q504 DNL BFG35, Q505 BFG35, Q506 DNL BFG31, Q507 DNL J310, T201 CMC 2 mH, T202 CMC 2 mH, T203 DNL T1-6, T501 DNL T-622, T502 DNL T1-6, T503 CMC 2 mH, T504 DNL T1-6, U201 LM2941, U501 TPS7A4501

Commit message: big update supporting first PCB fab
Big changes to Artix-7 A35 FPGA on first PCB fab.
Renaming project to "KiwiSDR".
New thread priority scheme.
New eCPU stack checking code.
Many performance improvements.
GPS timing now adjusts XO frequency.
New SPI transfer integrity checking code.
Improved event recording debug facility.
Parts:
- removed C201, C203, C214: 470n/100, wrx-SM1206
- removed C202, C209, C213: 330u/35 EL, wrx-CAP_10x10
- removed C204, C205, C206, C207, C208: 100n/100, wrx-SM0805
- removed C210: 22u/25 TA, wrx-CAP_D
- removed C211: 1n, wrx-SM0402
- removed C212: 470n, wrx-SM0402
- removed C215, C216: DNL, wrx-SM1206
- removed D201: BR 0.5A 400V, wrx-TO269_AA
- removed D202: TVS 25VAC, wrx-SM0805
- removed F201, F202: PPTC 200 mA, wrx-SM1812
- removed G501, G502: 75V, wrx-GDT
- removed the J13 at (309.0, 85.0)
- removed J14, J25, J26: DNL BNC, wrx-BNC_SMA_NO_VIP
- removed J20, J21: TB_2, wrx-TB_2P_2_54MM
- removed J22: DC JACK 2.1MM, wrx-DC_JACK_2_1MM
- removed J23: DNL RJ45, wrx-RJ45_8
- removed J24: DNL TB_2, wrx-TB_2P_2_54MM
- removed L201: 100uH, wrx-SM1812
- removed R201: 680R, wrx-SM0805
- removed R202: 11K5, wrx-SM0805
- removed R203: 1K, wrx-SM0805
- removed R204, R205, R206, R207: 47R, wrx-SM0805
- removed R213, R214, R215: 0R, wrx-SM0805
- removed R216: 1K5, wrx-SM0805
- removed R217: DNL, wrx-SM0805
- removed T201, T202: CMC 2 mH, wrx-CMC
- removed T203: DNL T1-6, wrx-MCL_KK81
- removed TP201, TP202: TEST_POINT, wrx-TP_1250
- removed U201: LM2941, wrx-TO263
- added FID1: FIDUCIAL, kiwi-FIDUCIAL_2_SIDE, F.Cu at (139.0, 85.0)
- added FID2: FIDUCIAL, kiwi-FIDUCIAL_2_SIDE, F.Cu at (219.0, 53.0)
- added GFX1: LOGO, kiwi-KIWI_10MM, F.Cu at (96.0, 61.0)
- added GFX3: OSHW, kiwi-OSHW_6MM, F.Cu at (91.5, 78.0)
- added J10: DNL BNC, kiwi-BNC_SMA_NO_VIP, F.Cu at (222.0, 79.5)
- C501, C502, C506: footprint wrx-SM1206 -> kiwi-SM1206
- C503, C507, C508: value DNL -> 470n/100; footprint wrx-SM0805 -> kiwi-SM1206
- C504, C505: value DNL -> DNL 470n/100; footprint wrx-SM0805 -> kiwi-SM1206; moved to B.Cu
- C509, C510, C511, C512, C513, C514, C515, C516, C517, C518, C519, C520, C522, C523, C526, L501, L502, L503, L504, L505, L507, R502, R515, R516, R519, R520, R521, R522, R523, R524, R525: footprint wrx-SM0805 -> kiwi-SM0805
- C521: value 470n/100 -> DNL 100n/100; footprint wrx-SM1206 -> kiwi-SM0805
- C524, C525, C527: value DNL -> 1n/100; footprint wrx-SM0805 -> kiwi-SM0805
- EP501: footprint wrx-E_FIELD_PROBE -> kiwi-E_FIELD_PROBE
- J11: footprint wrx-RJ45_8 -> kiwi-RJ45_8
- J12: footprint wrx-TB_2P_2_54MM -> kiwi-TB_2P_2_54MM; moved to B.Cu
- J13: renamed from J10; footprint wrx-TB_2P_2_54MM -> kiwi-TB_2P_2_54MM; moved to B.Cu
- L506: footprint wrx-SM1812 -> kiwi-SM1812
- L508, L509, L510: value DNL FB 80Z -> FB 80Z; footprint wrx-SM0805 -> kiwi-SM0805
- Q501: footprint wrx-SOT23_DGS -> kiwi-SOT23_DGS
- Q502: value DNL J271 -> J271; footprint wrx-SOT23_DGS -> kiwi-SOT23_DGS
- Q503, Q506: value DNL BFG31 -> BFG31; footprint wrx-SOT223_EBEC -> kiwi-SOT223_EBEC
- Q504: value DNL BFG35 -> BFG35; footprint wrx-SOT223_EBEC -> kiwi-SOT223_EBEC
- Q505: footprint wrx-SOT223_EBEC -> kiwi-SOT223_EBEC
- Q507: footprint wrx-SOT23_DGS -> kiwi-SOT23_DGS; moved to B.Cu
- R501: value DNL -> 1M; footprint wrx-SM0805 -> kiwi-SM0805
- R503, R504: value DNL -> DNL 100R; footprint wrx-SM0805 -> kiwi-SM0805; moved to B.Cu
- R505: value 2K2 -> 100K; footprint wrx-SM0805 -> kiwi-SM0805
- R506: value 0R -> 2K2; footprint wrx-SM0805 -> kiwi-SM0805
- R507: value 10K -> 100K; footprint wrx-SM0402 -> kiwi-SM0805
- R508, R509: value DNL -> 470R; footprint wrx-SM0805 -> kiwi-SM0805
- R510: value 220R/0.5W -> 10R/0.66W; footprint wrx-SM0805 -> kiwi-SM1206
- R511: value 1M -> DNL 1M; footprint wrx-SM0805 -> kiwi-SM0805
- R512: value 1M -> 0R; footprint wrx-SM0805 -> kiwi-SM0805
- R513, R518: value 0R -> DNL 0R; footprint wrx-SM0805 -> kiwi-SM0805
- R514: value 680R -> 100R; footprint wrx-SM0805 -> kiwi-SM0805
- R517: value 47R -> DNL 47R; footprint wrx-SM0805 -> kiwi-SM0805
- T501, T502: footprint wrx-MCL_KK81 -> kiwi-MCL_KK81; moved to B.Cu
- T503: footprint wrx-CMC -> kiwi-CMC
- T504: footprint wrx-MCL_KK81 -> kiwi-MCL_KK81
- TP501, TP502: footprint wrx-TP_1250 -> kiwi-TP_1250
- U501: footprint wrx-SOT232_6 -> kiwi-SOT223_6
- moved J12 148.0 mm to (198.0, 70.0), turned to 270 degrees
- moved J13 138.9 mm to (207.0, 79.0), turned to 270 degrees
- moved R525 130.0 mm to (186.0, 74.0), turned to 90 degrees
- moved L506 128.9 mm to (191.0, 73.0), turned to 0 degrees
- moved C509 128.0 mm to (195.0, 54.0), turned to 90 degrees
- moved R522 127.5 mm to (201.0, 54.0), turned to 90 degrees
- moved T504 125.8 mm to (196.0, 80.0)
- moved C522 125.1 mm to (198.0, 54.0), turned to 90 degrees
- moved J11 124.6 mm to (214.0, 65.3)
- moved T503 123.0 mm to (198.0, 62.0)
- moved R524 118.8 mm to (203.0, 85.0)
- moved R523 118.8 mm to (203.0, 75.0)
- moved TP501 117.7 mm to (192.0, 53.0)
- moved R521 114.2 mm to (185.0, 60.0), turned to 90 degrees
- moved R520 113.9 mm to (185.0, 56.0), turned to 270 degrees
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Connections:
- net /Active_Antenna/14.55 renamed /14.55
- net /Active_Antenna/ANT2 renamed /ANT2
- net /Active_Antenna/ANT3 renamed /ANT3
- net /Active_Antenna/ANT4 renamed /ANT4
- net /Active_Antenna/B1H renamed /B1H
- net /Active_Antenna/B1L renamed /B1L
- net /Active_Antenna/B2H renamed /B2H
- net /Active_Antenna/B2L renamed /B2L
- net /Active_Antenna/BIAS renamed /BIAS
- net /Active_Antenna/BIAS+ renamed /BIAS+
- net /Active_Antenna/BIAS- renamed /BIAS-
- net /Active_Antenna/DCIN renamed /DCIN
- net /Active_Antenna/E1H renamed /E1H
- net /Active_Antenna/E1L renamed /E1L
- net /Active_Antenna/E2H renamed /E2H
- net /Active_Antenna/E2L renamed /E2L
- net /Active_Antenna/EPROBE renamed /EPROBE
- net /Active_Antenna/FB1 renamed /FB1
- net /Active_Antenna/FB2 renamed /FB2
- net /Active_Antenna/FB3 renamed /FB3
- net /Active_Antenna/JHI renamed /JHI
- net /Active_Antenna/JLO renamed /JLO
- net /Active_Antenna/NF1H renamed /NF1H
- net /Active_Antenna/NF1L renamed /NF1L
- net /Active_Antenna/NF2H renamed /NF2H
- net /Active_Antenna/NF2L renamed /NF2L
- net /Active_Antenna/NF3H renamed /NF3H
- net /Active_Antenna/NF3L renamed /NF3L
- net /Active_Antenna/THI renamed /THI
- net /Active_Antenna/TLO renamed /TLO
- net /Active_Antenna/TP renamed /TP
- net /Active_Antenna/VADJ renamed /VADJ
- C506 pad 2: /Active_Antenna/OUT -> /OUT
- C507 pad 2: /Active_Antenna/OUT -> /OUT
- C526 pad 2: /Active_Antenna/OUT -> /OUT
- C527 pad 2: /Active_Antenna/OUT -> /OUT
- J11 pad 1: /Active_Antenna/RX- -> /RX-
- J11 pad 2: /Active_Antenna/RX+ -> /RX+
- J11 pad 4: /Active_Antenna/RX+ -> /RX+
- J11 pad 5: /Active_Antenna/RX- -> /RX-
- J13 pad 1: /Active_Antenna/RX+ -> /RX+
- J13 pad 2: /Active_Antenna/RX- -> /RX-
- L506 pad 1: /Active_Antenna/OUT -> /OUT
- R523 pad 1: /Active_Antenna/RX+ -> /RX+
- R523 pad 2: /Active_Antenna/OUT -> /OUT
- R524 pad 1: /Active_Antenna/RX- -> /RX-
- R525 pad 2: /Active_Antenna/OUT -> /OUT
- T504 pad 1: /Active_Antenna/RX- -> GND
- T504 pad 3: /Active_Antenna/RX+ -> /OUT
- T504 pad 4: /Active_Antenna/OUT -> /RX+
- T504 pad 6: GND -> /RX-
Routing:
- net /14.55: track 0.00 -> 142.0 mm, vias 0 -> 19
- net GND: track 0.00 -> 90.6 mm, vias 0 -> 29
- net /RX-: track 0.00 -> 56.0 mm, vias 0 -> 2
- net /OUT: track 0.00 -> 40.2 mm
- net /JHI: track 0.00 -> 37.0 mm, vias 0 -> 1
- net /BIAS+: track 0.00 -> 37.0 mm
- net /JLO: track 0.00 -> 32.8 mm, vias 0 -> 1
- net /RX+: track 0.00 -> 31.9 mm
- net /EPROBE: track 0.00 -> 31.0 mm
- net /BIAS-: track 0.00 -> 26.8 mm
- net /E2L: track 0.00 -> 23.8 mm
- net /DCIN: track 0.00 -> 23.4 mm
- net /E1H: track 0.00 -> 23.0 mm
- net /ANT4: track 0.00 -> 19.7 mm
- net /NF3L: track 0.00 -> 19.6 mm
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- added copper zone on B.Cu, net /14.55
- added copper zone on B.Cu, net GND
- added copper zone on F.Cu, net GND
Other:
- board size 300 x 155 mm -> 138 x 38 mm
- board text added: "-"
- board text added: "14.5V"
- board text added: "ANT"
- board text added: "Active Antenna"
- board text added: "August 2015"
- board text added: "BIAS+"
- board text added: "DC"
- board text added: "GND"
- board text added: "KiwiSDR"
- board text added: "OSHW"
- board text added: "jks.com/kiwisdr"
- board text added: "©Point Reyes Ventures, LLC"
- board text added: "©Sonoran Radio Research"
- board text added: "©bluebison.net"

Commit message: v0.5 PCB with 5V DC input
Other:
- board text added: "© John Seamons, ZL/KF6VO"
- board text added: "© Sonoran Radio Research"
- board text removed: "©Point Reyes Ventures, LLC"
- board text removed: "©Sonoran Radio Research"
Changed lines of the file:
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@@
   )
   (setup
-    (last_trace_width 0.5)
+    (last_trace_width 1)
     (user_trace_width 0.15)
     (user_trace_width 0.2)
@@
     )
   )
-  (gr_text "©Point Reyes Ventures, LLC" (at 117 78) (layer F.SilkS)
+  (gr_text "© John Seamons, ZL/KF6VO" (at 117 78) (layer F.SilkS)
     (effects (font (size 1.5 1.2) (thickness 0.2)))
   )
@@
     (effects (font (size 1.5 1.2) (thickness 0.2)) (justify right))
   )
-  (gr_text "©Sonoran Radio Research" (at 118 75) (layer F.SilkS)
+  (gr_text "© Sonoran Radio Research" (at 117.5 75) (layer F.SilkS)
     (effects (font (size 1.5 1.2) (thickness 0.2)))
   )
@@
   (segment (start 145 77.09982) (end 144.90018 77) (width 0.25) (layer Top) (net 9))
   (segment (start 148 80.0348) (end 145 80.0348) (width 0.25) (layer Top) (net 9))
-  (segment (start 198 68.73) (end 196.27 68.73) (width 0.5) (layer Top) (net 10) (status 400000))
-  (segment (start 195 73) (end 193.125 73) (width 0.5) (layer Top) (net 10) (status 800000))
+  (segment (start 198 68.73) (end 196.27 68.73) (width 0.5) (layer Top) (net 10))
+  (segment (start 195 73) (end 193.125 73) (width 0.5) (layer Top) (net 10))
   (segment (start 195.5 72.5) (end 195 73) (width 0.5) (layer Top) (net 10))
   (segment (start 195.5 69.5) (end 195.5 72.5) (width 0.5) (layer Top) (net 10))
   (segment (start 196.27 68.73) (end 195.5 69.5) (width 0.5) (layer Top) (net 10))
-  (segment (start 186 74.9652) (end 186.4652 74.9652) (width 0.25) (layer Top) (net 10) (status C00000))
-  (segment (start 186.4652 74.9652) (end 187.25 75.75) (width 0.25) (layer Top) (net 10) (status 400000))
+  (segment (start 186 74.9652) (end 186.4652 74.9652) (width 0.25) (layer Top) (net 10))
+  (segment (start 186.4652 74.9652) (end 187.25 75.75) (width 0.25) (layer Top) (net 10))
   (segment (start 187.25 75.75) (end 190.75 75.75) (width 0.25) (layer Top) (net 10))
   (segment (start 190.75 75.75) (end 191 75.5) (width 0.25) (layer Top) (net 10))
   (segment (start 191 75.5) (end 191 73.25) (width 0.25) (layer Top) (net 10))
   (segment (start 191 73.25) (end 191.25 73) (width 0.25) (layer Top) (net 10))
-  (segment (start 191.25 73) (end 193.125 73) (width 0.25) (layer Top) (net 10) (status 800000))
+  (segment (start 191.25 73) (end 193.125 73) (width 0.25) (layer Top) (net 10))
   (segment (start 205.11 63.445) (end 197.305 63.445) (width 0.5) (layer Top) (net 10))
   (segment (start 196.73 64.02) (end 196.73 65.75) (width 0.5) (layer Top) (net 10))
@@
   (segment (start 168 69.9652) (end 165 69.9652) (width 0.25) (layer Top) (net 28))
   (segment (start 165 69.9652) (end 163.9652 71) (width 0.25) (layer Top) (net 28))
-  (segment (start 186 73.0348) (end 188.8402 73.0348) (width 0.25) (layer Top) (net 29) (status C00000))
-  (segment (start 188.8402 73.0348) (end 188.875 73) (width 0.25) (layer Top) (net 29) (status C00000))
-  (segment (start 184.25 73.0348) (end 186 73.0348) (width 0.25) (layer Top) (net 29) (status 800000))
-  (segment (start 183 73.0348) (end 184.25 73.0348) (width 0.25) (layer Top) (net 29) (status 400000))
+  (segment (start 186 73.0348) (end 188.8402 73.0348) (width 0.25) (layer Top) (net 29))
+  (segment (start 188.8402 73.0348) (end 188.875 73) (width 0.25) (layer Top) (net 29))
+  (segment (start 184.25 73.0348) (end 186 73.0348) (width 0.25) (layer Top) (net 29))
+  (segment (start 183 73.0348) (end 184.25 73.0348) (width 0.25) (layer Top) (net 29))
   (segment (start 184.25 73.0348) (end 184.2152 73.0348) (width 0.25) (layer Top) (net 29))
-  (segment (start 189.93 77.5) (end 189.97 77.46) (width 0.25) (layer Top) (net 29) (status C00000))
-  (segment (start 185.25 77.5) (end 189.93 77.5) (width 0.25) (layer Top) (net 29) (status 800000))
+  (segment (start 189.93 77.5) (end 189.97 77.46) (width 0.25) (layer Top) (net 29))
+  (segment (start 185.25 77.5) (end 189.93 77.5) (width 0.25) (layer Top) (net 29))
   (segment (start 184.4304 76.6804) (end 185.25 77.5) (width 0.25) (layer Top) (net 29))
   (segment (start 184.4304 73.25) (end 184.4304 76.6804) (width 0.25) (layer Top) (net 29))
@@
   (segment (start 211.73 77.73) (end 213.5 79.5) (width 0.5) (layer Top) (net 30))
   (segment (start 205.11 65.985) (end 205.11 68.525) (width 0.5) (layer Top) (net 30))
-  (segment (start 203.9652 85) (end 206.5 85) (width 0.5) (layer Top) (net 31) (status 400000))
+  (segment (start 203.9652 85) (end 206.5 85) (width 0.5) (layer Top) (net 31))
   (segment (start 206.5 85) (end 207.75 83.75) (width 0.5) (layer Top) (net 31))
   (segment (start 202.03 82.54) (end 206.54 82.54) (width 0.5) (layer Top) (net 31))
