File: pcb/active_antenna/ant.sch (KiCad schematic (older format))
At the start: 85 parts, among them J10 DNL BNC, J11 DNL RJ45, J12 DNL TB_2, J13 TB_2, Q501 J310, Q502 J271, Q503 BFG31, Q504 BFG35, Q505 BFG35, Q506 BFG31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

Commit message: v0.5 PCB with 5V DC input
Parts:
- J10: value DNL BNC -> SMA
- J11: value DNL RJ45 -> RJ45
- J12: value DNL TB_2 -> TB_2
- T503: symbol COMMON_MODE_CHOKE -> COMMON_MODE_CHOKE_ALT
Connections:
- net BIAS-: now also T503.2; no longer T503.4
- net DCIN: now also T503.4; no longer T503.2
Other:
- note added: "COAX OPTION USED"
Changed lines of the file:
@@
-EESchema Schematic File Version 2  date Saturday, September 05, 2015 09:33:01 AM
+EESchema Schematic File Version 2  date Friday, February 12, 2016 06:49:53 PM
 LIBS:kiwi
+LIBS:ant-cache
 EELAYER 27 0
 EELAYER END
@@
 Sheet 1 1
 Title "KiwiSDR - Active Antenna and Power Supply"
-Date "4 sep 2015"
-Rev "1.0"
-Comp "Point Reyes Ventures, LLC"
-Comment1 "August 2015"
+Date "12 feb 2016"
+Rev "1.1"
+Comp ""
+Comment1 "February 2016"
 Comment2 ""
 Comment3 ""
@@
 $EndComp
 $Comp
-L COMMON_MODE_CHOKE T503
+L COMMON_MODE_CHOKE_ALT T503
 U 1 1 54EFFF1D
 P 12850 3300
@@
 P 14500 3000
 F 0 "J12" H 14500 3300 50  0000 C CNN
-F 1 "DNL TB_2" H 14500 2700 50  0000 C CNN
+F 1 "TB_2" H 14500 2700 50  0000 C CNN
 F 2 "kiwi-TB_2P_2_54MM" H 14500 3000 60  0001 C CNN
 F 3 "~" H 14500 3000 60  0000 C CNN
@@
 Text Label 10650 2100 0    60   ~ 0
 VADJ
-Text Label 14100 4500 0    60   ~ 0
+Text Label 13650 4500 0    60   ~ 0
 RX+
-Text Label 14100 4900 0    60   ~ 0
+Text Label 13650 4900 0    60   ~ 0
 RX-
 Text Label 13050 3100 0    60   ~ 0
@@
 P 14700 3850
 F 0 "J11" V 15200 4050 50  0000 C CNN
-F 1 "DNL RJ45" V 14250 4000 50  0000 C CNN
+F 1 "RJ45" V 14250 4000 50  0000 C CNN
 F 2 "kiwi-RJ45_8" H 14700 3950 60  0001 C CNN
 F 3 "~" H 14700 3950 60  0000 C CNN
@@
 U 1 1 55762A64
 P 14500 4650
-F 0 "J10" H 14250 4600 60  0000 C CNN
-F 1 "DNL BNC" V 14610 4590 40  0000 C CNN
+F 0 "J10" H 14250 4600 50  0000 C CNN
+F 1 "SMA" V 14610 4590 40  0000 C CNN
 F 2 "kiwi-BNC_SMA_NO_VIP" H 14500 4650 60  0001 C CNN
 F 3 "~" H 14500 4650 60  0000 C CNN
@@
 NoConn ~ 7150 1600
 NoConn ~ 8150 1600
+Text Notes 13250 5600 0    100  ~ 0
+COAX OPTION USED
 $EndSCHEMATC
