File: pcb/active_antenna_comb/ant.sch (KiCad schematic (older format))
At the start: 0 parts

Commit message: v0.5 PCB with 5V DC input
Parts:
- added C501, C502, C503, C506, C507, C508: 470n/100, kiwi-SM1206, symbol C
- added C504, C505: DNL 470n/100, kiwi-SM1206, symbol C
- added C509: 100n/100, kiwi-SM0805, symbol C
- added C510, C520: 10u/25, kiwi-SM0805, symbol C
- added C511, C512, C513, C514, C515, C516, C517, C518, C519: DNL, kiwi-SM0805, symbol C
- added C521: DNL 100n/100, kiwi-SM0805, symbol C
- added C522, C523, C524, C525, C526, C527: 1n/100, kiwi-SM0805, symbol C
- added EP501: E_FIELD_PROBE, kiwi-E_FIELD_PROBE, symbol E_FIELD_PROBE
- added FID1, FID2: FIDUCIAL, kiwi-FIDUCIAL_2_SIDE, symbol FIDUCIAL
- added GFX1: LOGO, kiwi-KIWI_10MM, symbol GRAPHIC
- added GFX3: OSHW, kiwi-OSHW_6MM, symbol GRAPHIC
- added J10: DNL BNC, kiwi-BNC_SMA_NO_VIP, symbol COAX_CONN_3P
- added J11: DNL RJ45, kiwi-RJ45_8, symbol RJ45-NO-SHIELD
- added J12: DNL TB_2, kiwi-TB_2P_2_54MM, symbol TERM_BLOCK_2POS_H
- added J13: TB_2, kiwi-TB_2P_2_54MM, symbol TERM_BLOCK_2POS_H
- added L501, L502, L503, L504, L505: 0R, kiwi-SM0805, symbol COIL
- added L506: 100uH, kiwi-SM1812, symbol COIL
- added L507, L508, L509, L510: FB 80Z, kiwi-SM0805, symbol FERRITE_CHIP
- added Q501: J310, kiwi-SOT23_DGS, symbol N_JFET
- added Q502: J271, kiwi-SOT23_DGS, symbol P_JFET
- added Q503, Q506: BFG31, kiwi-SOT223_EBEC, symbol PNP_2E
- added Q504, Q505: BFG35, kiwi-SOT223_EBEC, symbol NPN_2E
- added Q507: DNL J310, kiwi-SOT23_DGS, symbol N_JFET
- added R501, R502: 1M, kiwi-SM0805, symbol R
- added R503, R504: DNL 100R, kiwi-SM0805, symbol R
- added R505, R507: 100K, kiwi-SM0805, symbol R
- added R506: 2K2, kiwi-SM0805, symbol R
- added R508, R509: 470R, kiwi-SM0805, symbol R
- added R510: 10R/0.66W, kiwi-SM1206, symbol R
- added R511: DNL 1M, kiwi-SM0805, symbol R
- added R512, R515, R516, R519, R523, R524: 0R, kiwi-SM0805, symbol R
- added R513, R518: DNL 0R, kiwi-SM0805, symbol R
- added R514: 100R, kiwi-SM0805, symbol R
- added R517: DNL 47R, kiwi-SM0805, symbol R
- added R520: 11K, kiwi-SM0805, symbol R
- added R521: 1K, kiwi-SM0805, symbol R
- added R522: DNL, kiwi-SM0805, symbol R
- added R525: 1K5, kiwi-SM0805, symbol R
- added T501: DNL T-622, kiwi-MCL_KK81, symbol T-622
- added T502: DNL T1-6, kiwi-MCL_KK81, symbol T1-6_SPLIT
- added T503: CMC 2 mH, kiwi-CMC, symbol COMMON_MODE_CHOKE
- added T504: DNL T1-6, kiwi-MCL_KK81, symbol T1-6
- added TP501, TP502: TEST_POINT, kiwi-TP_1250, symbol TEST_POINT
- added U501: TPS7A4501, kiwi-SOT232_6, symbol VREG_5PIN
Connections:
- new net 14.55: C520.1, Q504.C, Q505.C, R501.1, R503.1, R505.1, R508.1, R511.1, R515.1, R520.1, T501.3, T502.4, TP502.1, U501.4 (VOUT)
- new net ANT2: C511.2, L501.1, R519.1
- new net ANT3: C501.1, R519.2
- new net ANT4: C501.2, Q501.G, R501.2, R512.1
- new net B1H: L509.2, Q503.B
- new net B1L: L510.2, Q504.B
- new net B2H: L507.2, Q505.B
- new net B2L: L508.2, Q506.B
- new net BIAS: C521.1, Q502.G, R502.2, R511.2, R512.2
- new net BIAS+: J11.3 (gr), J11.6 (GR), J12.1, L506.2, R525.1, T503.3
- new net BIAS-: J11.7 (br), J11.8 (BR), J12.2, T503.4
- new net DCIN: C509.1, C510.1, C522.1, T503.2, TP501.1, U501.1 (ENA), U501.2 (VIN)
- new net E1H: L507.1, Q503.E1, Q503.E2, R508.2, R517.1
- new net E1L: L508.1, Q504.E1, Q504.E2, R509.1
- new net E2H: C506.1, C526.1, Q505.E1, Q505.E2, R510.1
- new net E2L: C507.1, C527.1, Q506.E1, Q506.E2, R510.2, R518.1
- new net EPROBE: C511.1, EP501.1, L501.2
- new net FB1: Q501.D, R515.2, T502.6
- new net FB2: Q502.D, Q507.G, R513.1, R516.2, T502.3
- new net FB3: Q507.D, T501.4
- new net GND: C504.1, C505.2, C509.2, C510.2, C520.2, C521.2, C522.2, Q503.C, Q506.C, Q507.S, R502.1, R504.1, R507.2, R509.2, R516.1, R518.2, R521.1, R522.2, R524.2, T502.1, T504.1, U501.3 (GND), U501.TAB
- new net JHI: C502.1, C508.1, C523.1, C524.1, Q501.S, R514.2, T501.1
- new net JLO: C503.1, C508.2, C524.2, C525.1, Q502.S, R513.2, R514.1, T501.2
- new net NF1H: C502.2, C512.1, C513.1, C523.2, L502.1
- new net NF1L: C503.2, C516.1, C517.1, C525.2, L504.1
- new net NF2H: C512.2, C513.2, C514.1, C515.1, L502.2, L503.1
- new net NF2L: C516.2, C517.2, C518.1, C519.1, L504.2, L505.1
- new net NF3H: C514.2, C515.2, L503.2, L509.1, R505.2, R506.1, R517.2
- new net NF3L: C518.2, C519.2, L505.2, L510.1, R506.2, R507.1
- new net OUT: C506.2, C507.2, C526.2, C527.2, L506.1, R523.2, R525.2, T504.3
- new net RX+: J10.1 (In), J11.2 (OR), J11.4 (BU), J13.1, R523.1, T504.4
- new net RX-: J10.2 (gnd), J10.3 (gnd), J11.1 (or), J11.5 (bu), J13.2, R524.1, T504.6
- new net THI: C505.1, R504.2, T501.6
- new net TLO: C504.2, R503.2, T501.5
- new net TP: R522.1, T503.1
- new net VADJ: R520.2, R521.2, U501.5 (ADJ)
- no-connect marks 0 -> 2
Other:
- note added: "*"
- note added: "* NB: drain (not source)\nconnected to ground"
- note added: "30 MHz LPF"
- note added: "BCB notch filters"
- note added: "CAT5\n\n0R\nDNL\nDNL\nDNL\n\nDNL\nT1-6\n\nOPT\nOPT"
- note added: "COAX\n\nDNL\n0R\n0R\n1K5\n\n100uH\nDNL\n\nDNL\nDNL"
- note added: "DC In\nTO INJ J24"
- note added: "PA0RDT\nMINI\nWHIP\n\n\n470n\nDNL\nDNL\nDNL\n470n\nDNL\nDNL\n470n\n1n\nDNL\nDNL\n1n\nDNL\n"
- note added: "PA0RDT\nMINI\nWHIP\n\n\nDNL\n1M\nDNL\nDNL\n2K2\n0R\n10K\nDNL\nDNL\n220R\n1M\n1M\n0R\n680R\n0R\n0R\n47R\n0R\n"
- note added: "PA0RDT\nMINI\nWHIP\n\n\nJ310\nDNL\nDNL\nDNL\nBFG35\nDNL\nDNL\n\nDNL\nDNL\nLOAD\nDNL\nDNL\nDNL\n"
- note added: "PART\n\nR522\nR523\nR524\nR525\n\nL506\nT504\n\nJ11\nJ12"
- note added: "PART\n\n\n\n\nC502\nC503\nC504\nC505\nC506\nC507\nC508\nC521\nC523\nC524\nC525\nC526\nC527\n"
- note added: "PART\n\n\n\n\nQ501\nQ502\nQ503\nQ504\nQ505\nQ506\nQ507\n\nT501\nT502\nL507\nL508\nL509\nL510\n"
- note added: "PART\n\n\n\n\nR501\nR502\nR503\nR504\nR505\nR506\nR507\nR508\nR509\nR510\nR511\nR512\nR513\nR514\nR515\nR516\nR517\nR518\n"
- note added: "RF Out, DC In\nTO INJ J23"
- note added: "RF Out\nDC In\nTO INJ J21"
- note added: "TRASK\nCOMP\nPUSH\nPULL\n\n1M\n1M\nDNL\nDNL\n100K\n2K2\n100K\n470R\n470R\n10R\nDNL\n0R\nDNL\n100R\n0R\n0R\nDNL\nDNL\n"
- note added: "TRASK\nCOMP\nPUSH\nPULL\n\n470n\n470n\nDNL\nDNL\n470n\n470n\n470n\nDNL\n1n\n1n\n1n\n1n\n1n\n"
- note added: "TRASK\nCOMP\nPUSH\nPULL\n\nJ310\nJ271\nBFG31\nBFG35\nBFG35\nBFG31\nDNL\n\nDNL\nDNL\nLOAD\nLOAD\nLOAD\nLOAD\n"
- note added: "TRASK\nNEG\nFEED\nBACK\n\n1M\n1M\n100R\n100R\n100K\n2K2\n100K\n470R\n470R\n10R\nDNL\n0R\nDNL\nDNL\nDNL\nDNL\nDNL\nDNL\n"
- note added: "TRASK\nNEG\nFEED\nBACK\n\n470n\n470n\n470n\n470n\n470n\n470n\nDNL\nDNL\n1n\nDNL\n1n\n1n\n1n\n"
- note added: "TRASK\nNEG\nFEED\nBACK\n\nJ310\nJ271\nBFG31\nBFG35\nBFG35\nBFG31\nJ310\n\nT-622\nT1-6\nLOAD\nLOAD\nLOAD\nLOAD\n"
- note added: "Vin max 20V\n< 200 mV dropout\n35 nV/rHz noise\nreverse Vin protection"
