File: pcb/active_antenna_pwr/pwr.kicad_pcb (KiCad board)
At the start: 2 copper layers, 99 x 60 mm, 59 parts, among them J20 DNL TB_2, J21 DNL RJ45, J22 TB_2, J23 DNL BNC, J24 TB_2, J25 DNL BNC, J26 TB_2, J27 DNL TB_2, J28 DC JACK 2.1MM, Q201 MMBT4401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

Commit message: v0.5 PCB with 5V DC input
Parts:
- removed C218: 330u/35 EL, kiwi-CAP_10x10
- added C202: 470n/100, kiwi-SM1206, F.Cu at (212.5, 203.2)
- added C213: 1n/100, kiwi-SM0805, F.Cu at (212.2, 199.5)
- added D203: TVS 3.3V, kiwi-SOD323, F.Cu at (202.8, 121.8)
- added D204: TVS 3.3V, kiwi-SOD323, F.Cu at (202.5, 125.5)
- added J26: TB_2, kiwi-TB_2P_2_54MM, F.Cu at (191.5, 125.2)
- added R212: DNL, kiwi-SM0805, F.Cu at (212.1, 190.1)
- C215, C216: value DNL -> 470n/100
- J20: value DNL TB_2 -> TB_2
- J21: value DNL RJ45 -> RJ45
- J23, J25: value DNL BNC -> SMA
- J27: value DNL TB_2 -> SMA; footprint kiwi-TB_2P_2_54MM -> kiwi-BNC_SMA_NO_VIP
- L202: value 120mH 60mA -> 20mH 1A; footprint kiwi-INDUCTOR_12x12 -> kiwi-CMC_22x22
- R214, R215: value 0R -> DNL
- T203: value DNL T1-6 -> T-622
- moved J27 31.2 mm to (177.2, 122.8), turned to 270 degrees
- moved L202 8.25 mm to (154.2, 159.8)
- renumbered J26 to J28, J28 to J29
Connections:
- net /Power_Injector/AC3 renamed /AC3
- net /Power_Injector/AC4 renamed /AC4
- net /Power_Injector/AC5 renamed /AC5
- net /Power_Injector/BIAS+ renamed /BIAS+
- net /Power_Injector/BIAS- renamed /BIAS-
- net /Power_Injector/SNB renamed /SNB
- net /Power_Injector/SNB1 renamed /SNB1
- net /Power_Injector/SNB2 renamed /SNB2
- net /Power_Injector/SNB3 renamed /SNB3
- net /Power_Injector/SNB4 renamed /SNB4
- net /Power_Injector/TPG renamed /TPG
- net /Power_Injector/VADJ renamed /VADJ
- net /Power_Injector/VMULT renamed /VMULT
- net /Power_Injector/VOUT3 renamed /VOUT3
- C206 pad 1: /Power_Injector/VIN -> /VIN
- C208 pad 1: /Power_Injector/VIN -> /VIN
- C209 pad 1: /Power_Injector/VIN -> /VIN
- C214 pad 1: /Power_Injector/VIN -> /VIN
- C215 pad 2: /Power_Injector/AC2 -> /AC2
- C216 pad 2: /Power_Injector/AC2 -> /AC2
- D201 pad 3: /Power_Injector/VIN -> /VIN
- D202 pad 1: /Power_Injector/AC2 -> /AC2
- F201 pad 2: /Power_Injector/VOUT1 -> /VOUT1
- F202 pad 2: /Power_Injector/AC1 -> /AC1
- J21 pad 1: /Power_Injector/ANT- -> /ANT-
- J21 pad 2: /Power_Injector/ANT+ -> /ANT+
- J21 pad 4: /Power_Injector/ANT+ -> /ANT+
- J21 pad 5: /Power_Injector/ANT- -> /ANT-
- J22 pad 1: /Power_Injector/ANT+ -> /ANT+
- J22 pad 2: /Power_Injector/ANT- -> /ANT-
- J23 pad 1: /Power_Injector/ANT+ -> /ANT+
- J23 pad 2: /Power_Injector/ANT- -> /ANT-
- J23 pad 3: /Power_Injector/ANT- -> /ANT-
- J24 pad 1: /Power_Injector/RX+ -> /RX1+
- J24 pad 2: /Power_Injector/RX- -> /RX1-
- J25 pad 1: /Power_Injector/RX+ -> /RX1+
- J25 pad 2: /Power_Injector/RX- -> /RX1-
- J25 pad 3: /Power_Injector/RX- -> /RX1-
- J27 pad 1: /Power_Injector/AC1 -> /RX2+
- J27 pad 2: /Power_Injector/AC2 -> /RX2-
- J28 pad 1: GND -> N-000006
- J28 pad 2: GND -> N-000006
- J29 pad 1: /Power_Injector/AC1 -> /AC1
- J29 pad 2: /Power_Injector/AC2 -> /AC2
- J29 pad 3: /Power_Injector/AC2 -> /AC2
- L201 pad 1: /Power_Injector/RX+ -> /ANT+
- L202 pad 1: /Power_Injector/VOUT1 -> /VOUT2
- L202 pad 2: /Power_Injector/VOUT2 -> /VOUT1
- Q201 pad E: /Power_Injector/VOUT2 -> /VOUT2
- R205 pad 1: /Power_Injector/VIN -> /VIN
- R213 pad 1: /Power_Injector/ANT+ -> GND
- R213 pad 2: /Power_Injector/RX+ -> /ANT-
- R214 pad 1: /Power_Injector/ANT- -> /CPL
- R214 pad 2: /Power_Injector/RX- -> /RX1+
- R215 pad 2: /Power_Injector/RX- -> /RX1-
- R216 pad 2: /Power_Injector/RX+ -> /ANT+
- T202 pad 3: /Power_Injector/AC2 -> /AC2
- T203 pad 1: /Power_Injector/RX- -> /CPL
- T203 pad 2: (no net) -> /RX1+
- T203 pad 3: /Power_Injector/RX+ -> /RX2+
- T203 pad 4: /Power_Injector/ANT+ -> /RX2-
- T203 pad 5: (no net) -> /RX1-
- T203 pad 6: /Power_Injector/ANT- -> /ANT-
- TP201 pad 1: /Power_Injector/VIN -> /VIN
- TP202 pad 1: /Power_Injector/VOUT1 -> /VOUT1
- U201 pad 2: /Power_Injector/VIN -> GND
- U201 pad 4: /Power_Injector/VIN -> /VIN
Routing:
- net /Power_Injector/VIN: track 56.9 -> 0.00 mm
- net /VIN: track 0.00 -> 54.4 mm
- net /Power_Injector/ANT+: track 51.9 -> 0.00 mm
- net /ANT+: track 0.00 -> 51.9 mm
- net /Power_Injector/ANT-: track 50.6 -> 0.00 mm
- net /ANT-: track 0.00 -> 50.6 mm
- net /Power_Injector/AC2: track 49.1 -> 0.00 mm, vias 2 -> 0
- net /AC2: track 0.00 -> 49.1 mm, vias 0 -> 2
- net /Power_Injector/VOUT2: track 43.5 -> 0.00 mm
- net /VOUT2: track 0.00 -> 43.5 mm
- net /Power_Injector/AC1: track 36.9 -> 0.00 mm
- net /AC1: track 0.00 -> 36.9 mm
- net /VOUT1: track 0.00 -> 29.3 mm
- net /Power_Injector/VOUT1: track 29.3 -> 0.00 mm
- net /RX1-: track 0.00 -> 19.8 mm
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Other:
- board text added: "© John Seamons, ZL/KF6VO"
- board text removed: "©Point Reyes Ventures, LLC"
