File: pcb/active_antenna_pwr/pwr.sch (KiCad schematic (older format))
At the start: 59 parts, among them J20 DNL TB_2, J21 DNL RJ45, J22 TB_2, J23 DNL BNC, J24 TB_2, J25 DNL BNC, J26 TB_2, J27 DNL TB_2, J28 DC JACK 2.1MM, Q201 MMBT4401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

Commit message: v0.5 PCB with 5V DC input
Parts:
- removed C218: 330u/35 EL, kiwi-CAP_10x10, symbol CP1
- removed J27: DNL TB_2, kiwi-TB_2P_2_54MM, symbol TERM_BLOCK_2POS
- removed L202: 120mH 60mA, kiwi-INDUCTOR_12x12, symbol COIL
- removed R214: 0R, kiwi-SM0805, symbol R
- removed T203: DNL T1-6, kiwi-MCL_KK81, symbol T1-6
- added C202: 470n/100, kiwi-SM1206, symbol C
- added C213: 1n/100, kiwi-SM0805, symbol C
- added D203, D204: TVS 3.3V, kiwi-SOD323, symbol TVS
- added J26: TB_2, kiwi-TB_2P_2_54MM, symbol TERM_BLOCK_2POS
- added J27: SMA, kiwi-BNC_SMA_NO_VIP, symbol COAX_CONN_3P
- added L202: 20mH 1A, kiwi-CMC_22x22, symbol COMMON_MODE_CHOKE_ALT
- added R212, R215: DNL, kiwi-SM0805, symbol R
- added T203: T-622, kiwi-MCL_KK81, symbol T-622_ALT
- C215, C216: value DNL -> 470n/100
- J20: value DNL TB_2 -> TB_2
- J21: value DNL RJ45 -> RJ45
- J23, J25: value DNL BNC -> SMA
- J29: renamed from J28; value DC JACK 2.1MM -> POWER JACK 2.1MM
- R214: renamed from R213; value 0R -> DNL
- renumbered J26 to J28, R215 to R213
Connections:
- net ANT+: now also L201.1, R216.2, C202.1, C213.1, D203.2, D204.2, R212.1; no longer R214.1
- net ANT-: now also R213.2, D203.1, D204.1, T203.6
- net GND: now also R215.1
- net VOUT1: now also L202.2, L202.3
- net VOUT2: now also L202.1, L202.4
- net RX+ renamed RX1+
- net RX1+: now also T203.2; no longer L201.1, R216.2
- net RX- renamed RX1-
- net RX1-: now also R215.2, T203.5; no longer R213.2
- new net CPL: C202.2, C213.2, R212.2, R214.1, T203.1
- new net RX2+: J26.1, J27.1 (In), T203.3
- new net RX2-: J26.2, J27.2 (gnd), J27.3 (gnd), T203.4
Other:
- note added: "50/60 Hz LPF\nFc <= 30 Hz"
- note added: "CAT5\n\n\n\nDNL\nDNL\n\n0R\nDNL\nDNL\nDNL\nDNL\n0R\n\nT-622\nDNL\n"
- note added: "COAX BRAID-BREAKER OPTION USED"
- note added: "COAX\nBRAID-\nBREAKER\n\n470n\n1n\n\nDNL\n0R\nDNL\nDNL\n1K5\nDNL\n\nT-622\n100uH\n"
- note added: "COAX\n\n\n\n470n\n1n\n\nDNL\n0R\n0R\n0R\n1K5\nDNL\n\nDNL\n100uH\n"
- note added: "PART\n\n\n\nC202\nC213\n\nR212\nR213\nR214\nR215\nR216\nR217\n\nT203\nL201\n"
- note added: "TO ANT J13"
- note added: "TO RECEIVER #1 J1"
- note added: "TO RECEIVER #2 J1"
- note removed: "50/60 Hz LPF\nFc = 25 Hz"
- note removed: "CAT5\n\nDNL\nDNL\nDNL\nDNL\n0R\n\nT1-6\nDNL\n\nOPT\nOPT"
- note removed: "COAX\n\n0R\n0R\n0R\n1K5\nDNL\n\nDNL\n100uH\n\nDNL\nDNL"
- note removed: "PART\n\nR213\nR214\nR215\nR216\nR217\n\nT203\nL201\n\nJ23\nJ24\n"
- note removed: "TO RECEIVER J1"
- moved on the sheet: C209, C210, C211, C212, C214, C217, J20, J21, J22, J23, J24, J25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
